File: ESP-DEVKIT-MINI.kicad_sch (KiCad schematic)
At the start: 45 parts, among them J1 Conn_01x22_Pin, J2 Conn_01x22_Pin, J3 USB_C_Receptacle_USB2.0, J4 USB_B_Mini, J5 USB_B_Micro, Q1 L8050QLT1G, Q2 L8050QLT1G, SW1 SW_Omron_B3FS, SW2 SW_Omron_B3FS, U1 ESP32-S3-MINI-1-N8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

Commit message: Done
Connections:
- net GND: now also D3.1 (K)
Changed lines of the file:
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@@
+    )
+  )
+  (symbol (lib_id "PCM_4ms_Power-symbol:GND") (at 246.38 111.76 0) (unit 1)
+    (in_bom yes) (on_board yes) (dnp no) (fields_autoplaced)
+    (property "Reference" "#PWR021" (at 246.38 118.11 0)
+      (effects (font (size 1.27 1.27)) hide)
+    )
+    (property "Value" "GND" (at 246.38 116.84 0)
+      (effects (font (size 1.27 1.27)))
+    )
+    (property "Footprint" "" (at 246.38 111.76 0)
+      (effects (font (size 1.27 1.27)) hide)
+    )
+    (property "Datasheet" "" (at 246.38 111.76 0)
+      (effects (font (size 1.27 1.27)) hide)
+    )
+    (pin "1")
+    (instances
+      (project "ESP-DEVKIT-MINI"
+        (path "/473b80a5-6d9c-42aa-9c06-31a8cb982a54"
+          (reference "#PWR021") (unit 1)
+        )
+      )
     )
   )
